File: pcb/camera2/kicad/camera2.kicad_pcb (KiCad board)
At the start: 4 copper layers, 96.5 x 45.7 mm, 142 parts

Commit message: close to finishing netlist
Parts:
- removed REG0: , gen:7b67745b4d523e87fae434cdb8f46b54d22e1bc4395fdb8e73632e915883351d
- removed REG0C1, REG0C2: , gen:b8abd8cbc0b572999067c05d37fd407a90732e005a9769bc0f5d9b36d5f7537a
- removed REG1: , gen:798cf5bb0b3169533f5ca04ecb4ee99ae7bea0b47d3b6b0eac8ced07210df3aa
- removed REG2: , gen:6bc819ec539c21ef6344b6fd02be2ed3f4459069e5b504ecb87402b55c84b9f4
- removed REG3: , gen:817c1b12dae0694d00766759c3a729f1e099230e7310e0e9cf5cf1b3dbba25eb
- added vcc1_2_1C1: , gen:b8abd8cbc0b572999067c05d37fd407a90732e005a9769bc0f5d9b36d5f7537a, B.Cu at (111.8, 129.5)
- added vcc1_2_1C2: , gen:b8abd8cbc0b572999067c05d37fd407a90732e005a9769bc0f5d9b36d5f7537a, B.Cu at (116.8, 129.5)
- added vcc1_2_1U: , gen:4c0c04bd9660d62d02ba1b1137e43207b220c0f554dd932df5ec1e7ae8645dea, B.Cu at (114.3, 129.5)
- added vcc1_2_2U: , gen:4c0c04bd9660d62d02ba1b1137e43207b220c0f554dd932df5ec1e7ae8645dea, F.Cu at (177.8, 127.0)
- added vcc1_8U: , gen:26b8ae6ee31ef39667a5c9bab90434ae8d2e880264086e6bbcf67fafc1e30726, F.Cu at (149.9, 132.1)
- added vcc1_8_1U: , gen:26b8ae6ee31ef39667a5c9bab90434ae8d2e880264086e6bbcf67fafc1e30726, F.Cu at (91.4, 94.0)
- added vcc1_8_2C1: , gen:b8abd8cbc0b572999067c05d37fd407a90732e005a9769bc0f5d9b36d5f7537a, F.Cu at (213.4, 106.7)
- added vcc1_8_2C2: , gen:b8abd8cbc0b572999067c05d37fd407a90732e005a9769bc0f5d9b36d5f7537a, F.Cu at (218.4, 106.7)
- added vcc1_8_2U: , gen:26b8ae6ee31ef39667a5c9bab90434ae8d2e880264086e6bbcf67fafc1e30726, F.Cu at (215.9, 106.7)
- added vcc2_8C1: , gen:b8abd8cbc0b572999067c05d37fd407a90732e005a9769bc0f5d9b36d5f7537a, F.Cu at (147.3, 139.7)
- added vcc2_8C2: , gen:b8abd8cbc0b572999067c05d37fd407a90732e005a9769bc0f5d9b36d5f7537a, F.Cu at (152.4, 139.7)
- added vcc2_8U: , gen:fcc43d3bb1e6c2b6d917c0ea189430b092db7e0e9599257b1d9363923f608f14, F.Cu at (149.9, 139.7)
- added vcc3_0C1: , gen:b8abd8cbc0b572999067c05d37fd407a90732e005a9769bc0f5d9b36d5f7537a, F.Cu at (147.3, 147.3)
- added vcc3_0C2: , gen:b8abd8cbc0b572999067c05d37fd407a90732e005a9769bc0f5d9b36d5f7537a, F.Cu at (152.4, 147.3)
- added vcc3_0U: , gen:3bf6bb3add1bc1702bcd89948a5346a6e8cc093cbec858ea354b6d73d8980c49, F.Cu at (149.9, 147.3)
- added vcc3_0_1aC1: , gen:b8abd8cbc0b572999067c05d37fd407a90732e005a9769bc0f5d9b36d5f7537a, F.Cu at (88.9, 101.6)
- added vcc3_0_1aC2: , gen:b8abd8cbc0b572999067c05d37fd407a90732e005a9769bc0f5d9b36d5f7537a, F.Cu at (94.0, 101.6)
- added vcc3_0_1aU: , gen:3bf6bb3add1bc1702bcd89948a5346a6e8cc093cbec858ea354b6d73d8980c49, F.Cu at (91.4, 101.6)
- added vcc3_0_1bC1: , gen:b8abd8cbc0b572999067c05d37fd407a90732e005a9769bc0f5d9b36d5f7537a, F.Cu at (88.9, 109.2)
- added vcc3_0_1bC2: , gen:b8abd8cbc0b572999067c05d37fd407a90732e005a9769bc0f5d9b36d5f7537a, F.Cu at (94.0, 109.2)
- added vcc3_0_1bU: , gen:3bf6bb3add1bc1702bcd89948a5346a6e8cc093cbec858ea354b6d73d8980c49, F.Cu at (91.4, 109.2)
- added vcc3_0_2aC1: , gen:b8abd8cbc0b572999067c05d37fd407a90732e005a9769bc0f5d9b36d5f7537a, F.Cu at (213.4, 111.8)
- added vcc3_0_2aC2: , gen:b8abd8cbc0b572999067c05d37fd407a90732e005a9769bc0f5d9b36d5f7537a, F.Cu at (218.4, 111.8)
- added vcc3_0_2aU: , gen:3bf6bb3add1bc1702bcd89948a5346a6e8cc093cbec858ea354b6d73d8980c49, F.Cu at (215.9, 111.8)
- added vcc3_0_2bC1: , gen:b8abd8cbc0b572999067c05d37fd407a90732e005a9769bc0f5d9b36d5f7537a, F.Cu at (213.4, 116.8)
- added vcc3_0_2bC2: , gen:b8abd8cbc0b572999067c05d37fd407a90732e005a9769bc0f5d9b36d5f7537a, F.Cu at (218.4, 116.8)
- added vcc3_0_2bU: , gen:3bf6bb3add1bc1702bcd89948a5346a6e8cc093cbec858ea354b6d73d8980c49, F.Cu at (215.9, 116.8)
- B1, B10, B11, B15, B16, B17, B18, B19, B2, B20, B3, B4, B5, B6: footprint gen:499eb9275f53d39e8577307f805591431933e719fae192caf99d98aedcaee8aa -> gen:10ef96ba47ea821d370b2a1bfc3c3d814d7b338ee5b7ffa7a1f1d8c85d540e15
- IU3: footprint gen:eae6644e6b99af62deb74575fada904c5eece19a089fdb5d682cd29a528e43eb -> gen:ecc3b38187244d7633c640e655a8cec4f7c60211ad356d0b640b7827240d3be2
- MU1: footprint gen:8eebdf892b6f01e0d95a0c2299292ab3ec84d1b3707fa7ee95a6b86d4bb590c8 -> gen:9732419ddc38cd15a31e7c7960d0cee90905f01e9fbef09742a246810e6cbe16
- moved vcc1_2_2C2 76.9 mm to (180.3, 127.0), turned to 270 degrees
- moved vcc1_2_2C1 75.4 mm to (175.3, 127.0), turned to 270 degrees
- moved vcc1_8C1 69.6 mm to (147.3, 132.1), turned to 270 degrees
- moved vcc1_8C2 68.9 mm to (152.4, 132.1), turned to 270 degrees
- moved vcc1_8_1C1 62.1 mm to (88.9, 94.0), turned to 270 degrees
- moved vcc1_8_1C2 57.0 mm to (94.0, 94.0), turned to 270 degrees
- moved C1C21 34.2 mm to (43.2, 73.7)
- moved C1C41 34.2 mm to (48.3, 73.7)
- moved C1C11 34.2 mm to (40.6, 73.7)
- moved C1C31 34.2 mm to (45.7, 73.7)
- moved C1C33 34.2 mm to (45.7, 78.7)
- moved C1C51 34.2 mm to (50.8, 73.7)
- moved C1C61 34.2 mm to (53.3, 73.7)
- moved C1C63 34.2 mm to (53.3, 78.7)
- moved C1C20 34.2 mm to (43.2, 71.1)
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- renumbered REG1C1 to vcc1_2_2C1, REG1C2 to vcc1_2_2C2, REG2C1 to vcc1_8C1, REG2C2 to vcc1_8C2, REG3C1 to vcc1_8_1C1, REG3C2 to vcc1_8_1C2
Connections:
- net pwm1 renamed led_pwm1
- net pwm2 renamed led_pwm2
- net pwm3 renamed led_pwm3
- C1C10 pad 1: vcc1_8 -> vcc1_8_1
- C1C11 pad 1: vcc1_8 -> vcc1_8_1
- C1C12 pad 1: vcc1_8 -> vcc1_8_1
- C1C20 pad 1: vcc1_8 -> vcc1_8_1
- C1C21 pad 1: vcc1_8 -> vcc1_8_1
- C1C30 pad 1: vcc3_0 -> vcc3_0_1a
- C1C31 pad 1: vcc3_0 -> vcc3_0_1a
- C1C32 pad 1: vcc3_0 -> vcc3_0_1a
- C1C33 pad 1: vcc3_0 -> vcc3_0_1a
- C1C40 pad 1: vcc3_0 -> vcc3_0_1a
- C1C41 pad 1: vcc3_0 -> vcc3_0_1a
- C1C50 pad 1: vcc3_0 -> vcc3_0_1a
- C1C51 pad 1: vcc3_0 -> vcc3_0_1a
- C1FB1 pad 1: vcc3_0 -> vcc3_0_1b
- C1U1 pad 1: vcc3_0 -> vcc3_0_1a
- C1U1 pad 19: vcc3_0 -> vcc3_0_1a
- C1U1 pad 22: vcc1_8 -> vcc1_8_1
- C1U1 pad 26: vcc1_8 -> vcc1_8_1
- C1U1 pad 29: vcc3_0 -> vcc3_0_1a
- C1U1 pad 36: vcc3_0 -> vcc3_0_1a
- C1U1 pad 6: vcc1_8 -> vcc1_8_1
- C2C10 pad 1: vcc1_8 -> vcc1_8_2
- C2C11 pad 1: vcc1_8 -> vcc1_8_2
- C2C12 pad 1: vcc1_8 -> vcc1_8_2
- C2C20 pad 1: vcc1_8 -> vcc1_8_2
- C2C21 pad 1: vcc1_8 -> vcc1_8_2
- C2C30 pad 1: vcc3_0 -> vcc3_0_2a
- C2C31 pad 1: vcc3_0 -> vcc3_0_2a
- C2C32 pad 1: vcc3_0 -> vcc3_0_2a
- C2C33 pad 1: vcc3_0 -> vcc3_0_2a
- C2C40 pad 1: vcc3_0 -> vcc3_0_2a
- C2C41 pad 1: vcc3_0 -> vcc3_0_2a
- C2C50 pad 1: vcc3_0 -> vcc3_0_2a
- C2C51 pad 1: vcc3_0 -> vcc3_0_2a
- C2FB1 pad 1: vcc3_0 -> vcc3_0_2b
- C2U1 pad 1: vcc3_0 -> vcc3_0_2a
- C2U1 pad 19: vcc3_0 -> vcc3_0_2a
- C2U1 pad 22: vcc1_8 -> vcc1_8_2
- C2U1 pad 26: vcc1_8 -> vcc1_8_2
- C2U1 pad 29: vcc3_0 -> vcc3_0_2a
- C2U1 pad 36: vcc3_0 -> vcc3_0_2a
- C2U1 pad 6: vcc1_8 -> vcc1_8_2
- D0U pad 8: vcc3_0 -> vcc3_3in
- D1U pad 8: vcc3_0 -> vcc3_3in
- D2U pad 8: vcc3_0 -> vcc3_3in
- D3U pad 8: vcc3_0 -> vcc3_3in
- IU3 pad 35: pwm0 -> led_pwm0
- T1U pad 7: vcc1_2 -> vcc1_2_1
- T2U pad 7: vcc1_2 -> vcc1_2_2
- U2 pad 53: _U2_53_IO1_53 -> temp_bus
- U2 pad 54: _U2_54_IO1_54 -> led_pwm0
- U2 pad 55: _U2_55_IO1_55 -> led_pwm0
- U2 pad 56: _U2_56_IO1_56 -> led_pwm0
- U2 pad 58: _U2_58_IO1_58 -> led_pwm0
- vcc1_2_2C2 pad 1: vcc1_8 -> vcc1_2_2
- vcc1_8C2 pad 1: vcc1_2 -> vcc1_8
- vcc1_8_1C2 pad 1: vcc2_8 -> vcc1_8_1
Routing:
- net vcc3_0: track 8.77 -> 3.15 mm, vias 8 -> 2
- net vcc1_8: track 5.21 -> 0.00 mm, vias 5 -> 0
- net vcc3_0_1a: track 0.00 -> 3.67 mm, vias 0 -> 4
- net vcc1_8_1: track 0.00 -> 3.19 mm, vias 0 -> 3
- net vcc1_8_2: track 0.00 -> 2.02 mm, vias 0 -> 2
- net vcc3_0_2a: track 0.00 -> 1.95 mm, vias 0 -> 2
- net vcc1_2: track 1.31 -> 0.00 mm, vias 2 -> 0
- net vcc1_2_1: track 0.00 -> 0.66 mm, vias 0 -> 1
- net vcc1_2_2: track 0.00 -> 0.65 mm, vias 0 -> 1
- added copper zone on In1.Cu, net vcc3_3in
- removed copper zone on In1.Cu, net vcc3_0

Commit message: more work on netlist
Parts:
- removed ID4C, ID5C, ID6C, ID7C: , gen:b8abd8cbc0b572999067c05d37fd407a90732e005a9769bc0f5d9b36d5f7537a
- removed IL0, IL1, IL2, IL3: , gen:5ee2e2daf856c7b57c8b813aab30cc4a712b0ba6b927f36d7f82f0d8799f116d
- removed the vcc1_2_1U at (114.3, 129.5)
- removed the vcc1_2_2U at (177.8, 127.0)
- removed the vcc1_8U at (149.9, 132.1)
- removed the vcc1_8_1U at (91.4, 94.0)
- removed the vcc1_8_2U at (215.9, 106.7)
- removed the vcc2_8U at (149.9, 139.7)
- removed the vcc3_0U at (149.9, 147.3)
- removed the vcc3_0_1aU at (91.4, 101.6)
- removed the vcc3_0_1bU at (91.4, 109.2)
- removed the vcc3_0_2aU at (215.9, 111.8)
- removed the vcc3_0_2bU at (215.9, 116.8)
- added ID0C2: , gen:b8abd8cbc0b572999067c05d37fd407a90732e005a9769bc0f5d9b36d5f7537a, F.Cu at (154.1, 116.3)
- added ID0J: , gen:296adfb6ef4c709971068baccf341c4591f424b4dea6c069cef9fe0d7e190f60, F.Cu at (160.6, 118.7)
- added ID0L: , gen:da622f5a87a9fb4c0aae29dcedeb6324dab8b361c3014f17f52cf5734a2495b1, F.Cu at (137.1, 156.2)
- added ID1C2: , gen:b8abd8cbc0b572999067c05d37fd407a90732e005a9769bc0f5d9b36d5f7537a, F.Cu at (154.3, 118.0)
- added ID1J: , gen:296adfb6ef4c709971068baccf341c4591f424b4dea6c069cef9fe0d7e190f60, F.Cu at (160.7, 119.0)
- added ID1L: , gen:da622f5a87a9fb4c0aae29dcedeb6324dab8b361c3014f17f52cf5734a2495b1, F.Cu at (146.5, 157.9)
- added ID2C2: , gen:b8abd8cbc0b572999067c05d37fd407a90732e005a9769bc0f5d9b36d5f7537a, F.Cu at (154.7, 119.5)
- added ID2J: , gen:296adfb6ef4c709971068baccf341c4591f424b4dea6c069cef9fe0d7e190f60, F.Cu at (160.8, 119.4)
- added ID2L: , gen:da622f5a87a9fb4c0aae29dcedeb6324dab8b361c3014f17f52cf5734a2495b1, F.Cu at (155.1, 159.6)
- added ID3C2: , gen:b8abd8cbc0b572999067c05d37fd407a90732e005a9769bc0f5d9b36d5f7537a, F.Cu at (154.6, 121.1)
- added ID3J: , gen:296adfb6ef4c709971068baccf341c4591f424b4dea6c069cef9fe0d7e190f60, F.Cu at (160.8, 119.8)
- added ID3L: , gen:da622f5a87a9fb4c0aae29dcedeb6324dab8b361c3014f17f52cf5734a2495b1, F.Cu at (166.2, 162.6)
- added ID4D: , gen:7a59ddaa4fa6acd44dea9a71a48a5218831e1baf1b1d99cfe7246657470fcfd5, F.Cu at (141.1, 120.4)
- added ID5D: , gen:7a59ddaa4fa6acd44dea9a71a48a5218831e1baf1b1d99cfe7246657470fcfd5, F.Cu at (141.2, 117.8)
- added ID6D: , gen:7a59ddaa4fa6acd44dea9a71a48a5218831e1baf1b1d99cfe7246657470fcfd5, F.Cu at (141.5, 115.5)
- added ID7D: , gen:7a59ddaa4fa6acd44dea9a71a48a5218831e1baf1b1d99cfe7246657470fcfd5, F.Cu at (141.5, 113.3)
- added IR3: , gen:8b8e8cdd2a6c07e3e6c854f6b6a8f0d2287e4fa4909b824e776fd2ffcb4b4dd2, F.Cu at (149.9, 50.7)
- added vcc1_2_1U: , gen:b12d8ddcb22cae616881dc3cebe364fae9f00df16ee7f26dba84c179b2c59a7a, B.Cu at (114.3, 129.5)
- added vcc1_2_2U: , gen:b12d8ddcb22cae616881dc3cebe364fae9f00df16ee7f26dba84c179b2c59a7a, F.Cu at (177.8, 127.0)
- added vcc1_8U: , gen:ab734b132a751b905d3edc53450d623ac1384ebecf179d582a97cce317675793, F.Cu at (149.9, 50.8)
- added vcc1_8_1U: , gen:ab734b132a751b905d3edc53450d623ac1384ebecf179d582a97cce317675793, F.Cu at (91.4, 94.0)
- added vcc1_8_2U: , gen:ab734b132a751b905d3edc53450d623ac1384ebecf179d582a97cce317675793, F.Cu at (215.9, 106.7)
- added vcc2_8U: , gen:9f98c02c84ecd017867f5772ce06c41d0a832907966eb404fb4fbe7e6de904ad, F.Cu at (149.9, 58.5)
- added vcc3_0U: , gen:5300aaef9b9873e2073228bd9afa7c5cc2a8c7aa25bd73c625701e2266760cb5, F.Cu at (149.9, 66.1)
- added vcc3_0_1aU: , gen:5300aaef9b9873e2073228bd9afa7c5cc2a8c7aa25bd73c625701e2266760cb5, F.Cu at (91.4, 101.6)
- added vcc3_0_1bU: , gen:5300aaef9b9873e2073228bd9afa7c5cc2a8c7aa25bd73c625701e2266760cb5, F.Cu at (91.4, 109.2)
- added vcc3_0_2aU: , gen:5300aaef9b9873e2073228bd9afa7c5cc2a8c7aa25bd73c625701e2266760cb5, F.Cu at (215.9, 111.8)
- added vcc3_0_2bU: , gen:5300aaef9b9873e2073228bd9afa7c5cc2a8c7aa25bd73c625701e2266760cb5, F.Cu at (215.9, 116.8)
- B1, B10, B11, B15, B16, B17, B18, B19, B2, B20, B3, B4, B5, B6: footprint gen:10ef96ba47ea821d370b2a1bfc3c3d814d7b338ee5b7ffa7a1f1d8c85d540e15 -> gen:d8f50a25e8aff35263f8cecdeff9c4e270c76c16c279eea1f2c61de037ffe0fa
- C1U1, C2U1: footprint gen:b63fcc5f9d3775f8fe70cf3fb5d8b5f04a7eca08ac47608b5e89638e98bcb700 -> gen:1ad7109002e715198f83cca1ffc9049c8e5399a3842da71963adabba6beed15b
- IU3: footprint gen:ecc3b38187244d7633c640e655a8cec4f7c60211ad356d0b640b7827240d3be2 -> gen:7f2b3144da42c433b15ca783ca7830c64f1f439c0eded0fed474f7f4b6ae4199
- MU1: footprint gen:9732419ddc38cd15a31e7c7960d0cee90905f01e9fbef09742a246810e6cbe16 -> gen:118301f00dc3a559b9b2dce5a7b5f72bf6d5ed1b69630a5bdce773a57167cb56
- moved vcc1_8C1 81.3 mm to (147.3, 50.8)
- moved vcc1_8C2 81.3 mm to (152.4, 50.8)
- moved vcc3_0C1 81.2 mm to (147.3, 66.1)
- moved vcc3_0C2 81.2 mm to (152.4, 66.1)
- moved vcc2_8C1 81.2 mm to (147.3, 58.5)
- moved vcc2_8C2 81.2 mm to (152.4, 58.5)
- moved MU1 41.7 mm to (202.0, 35.1)
Connections:
- ID0C pad 1: vcc5in -> Icap0
- ID0R pad 1: vcc5in -> Icap0
- ID1C pad 1: vcc5in -> Icap1
- ID1R pad 1: vcc5in -> Icap1
- ID2C pad 1: vcc5in -> Icap2
- ID2R pad 1: vcc5in -> Icap2
- ID3C pad 1: vcc5in -> Icap3
- ID3R pad 1: vcc5in -> Icap3
- IU3 pad 10: vcc5in -> Icap3
- IU3 pad 18: vcc5in -> led_nSHDN
- IU3 pad 3: vcc5in -> Icap0
- IU3 pad 4: vcc5in -> Icap1
- IU3 pad 9: vcc5in -> Icap2
- U2 pad 55: led_pwm0 -> led_pwm1
- U2 pad 56: led_pwm0 -> led_pwm2
- U2 pad 58: led_pwm0 -> led_pwm3
- U2 pad 59: _U2_59_IO1_59 -> led_nSHDN
Other:
- board text removed: "1.2"
- board text removed: "1.8"
- board text removed: "2.8"

Commit message: tmp
Parts:
- moved ID0C 107.9 mm to (251.1, 147.1)
- moved ID0C2 107.9 mm to (258.1, 145.2)
- moved ID0J 107.9 mm to (264.6, 147.6)
- moved ID0R 107.9 mm to (254.7, 147.1)
- moved ID1C 107.9 mm to (251.3, 148.1)
- moved ID1J 107.9 mm to (264.7, 147.9)
- moved ID1R 107.9 mm to (254.8, 148.1)
- moved ID2C 107.9 mm to (251.1, 149.1)
- moved ID2C2 107.9 mm to (258.7, 148.3)
- moved ID2R 107.9 mm to (254.9, 149.1)
- moved ID3C 107.9 mm to (251.3, 149.9)
- moved ID3C2 107.9 mm to (258.6, 149.9)
- moved ID3J 107.9 mm to (264.8, 148.6)
- moved ID3R 107.9 mm to (254.9, 150.2)
- moved ID4D 107.9 mm to (245.1, 149.3)
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Routing:
- net C1trigger1: track 39.7 -> 5.45 mm
- net C1trigger2: track 37.7 -> 3.55 mm
- net C1trigger0: track 42.1 -> 8.06 mm
- net C1monitor0: track 36.7 -> 3.27 mm
- net C1monitor1: track 35.7 -> 2.90 mm
- net C1reset_n: track 34.7 -> 2.54 mm
- net C1_ss_n: track 33.7 -> 2.19 mm
- net C1MOSI: track 30.9 -> 1.80 mm
- net C1MISO: track 29.8 -> 1.45 mm
- net C1SCLK: track 28.8 -> 1.11 mm
- net T1_master_clk: track 30.4 -> 4.39 mm
- net T1_ss_n: track 72.4 -> 46.5 mm
- net T1_pwr_dwn_l: track 30.1 -> 4.30 mm
- net T1_reset_l: track 27.8 -> 2.78 mm
- net T1SCL: track 40.7 -> 17.7 mm
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
Commit message: the flippening
Parts:
- removed the B10C at (146.4, 92.6)
- removed the B11C at (155.3, 91.9)
- removed the B15C at (164.1, 98.0)
- removed the B16C at (160.0, 91.0)
- removed the B17C at (164.4, 92.7)
- removed the B18C at (161.6, 86.6)
- removed the B19C at (166.1, 88.5)
- removed the B1C at (120.0, 88.3)
- removed the B20C at (180.7, 89.4)
- removed the B2C at (134.7, 90.3)
- removed the B3C at (140.1, 87.0)
- removed the B4C at (137.4, 93.0)
- removed the B5C at (142.8, 89.9)
- removed the B6C at (140.2, 95.8)
- removed the D0U at (113.3, 84.3)
- removed the D1U at (109.7, 118.4)
- removed the D2U at (189.7, 118.5)
- removed the D3U at (186.3, 84.1)
- removed the ID0C at (251.1, 147.1)
- removed the ID0J at (264.6, 147.6)
- removed the ID0L at (137.1, 156.2)
- removed the ID0R at (254.7, 147.1)
- removed the ID1C at (251.3, 148.1)
- removed the ID1J at (264.7, 147.9)
- removed the ID1L at (146.5, 157.9)
- removed the ID1R at (254.8, 148.1)
- removed the ID2C at (251.1, 149.1)
- removed the ID2J at (264.8, 148.3)
- removed the ID2L at (155.1, 159.6)
- removed the ID2R at (254.9, 149.1)
- removed the ID3C at (251.3, 149.9)
- removed the ID3J at (264.8, 148.6)
- removed the ID3L at (166.2, 162.6)
- removed the ID3R at (254.9, 150.2)
- removed the ID4D at (245.1, 149.3)
- removed the ID5D at (245.2, 146.6)
- removed the ID6D at (245.5, 144.4)
- removed the ID7D at (245.5, 142.2)
- removed the IRT at (255.1, 136.2)
- removed the IU3C at (249.8, 141.8)
- removed the T1U at (118.4, 114.8)
- removed the T2U at (181.4, 114.8)
- removed the vcc1_2_1U at (114.3, 129.5)
- removed the vcc1_2_2U at (177.8, 127.0)
- removed the vcc1_8U at (149.9, 50.8)
- removed the vcc1_8_1U at (91.4, 94.0)
- removed the vcc1_8_2U at (215.9, 106.7)
- removed the vcc2_8U at (149.9, 58.5)
- removed the vcc3_0U at (149.9, 66.1)
- removed the vcc3_0_1aU at (91.4, 101.6)
- removed the vcc3_0_1bU at (91.4, 109.2)
- removed the vcc3_0_2aU at (215.9, 111.8)
- removed the vcc3_0_2bU at (215.9, 116.8)
- added B10C: , gen:15aef6ed4df9f5d238c1130cb8f0958fd2b96be76bbd888f3ba8bd3f59a98fb9, F.Cu at (146.4, 92.6)
- added B11C: , gen:15aef6ed4df9f5d238c1130cb8f0958fd2b96be76bbd888f3ba8bd3f59a98fb9, F.Cu at (155.3, 91.9)
- added B15C: , gen:15aef6ed4df9f5d238c1130cb8f0958fd2b96be76bbd888f3ba8bd3f59a98fb9, F.Cu at (164.1, 98.0)
- added B16C: , gen:15aef6ed4df9f5d238c1130cb8f0958fd2b96be76bbd888f3ba8bd3f59a98fb9, F.Cu at (160.0, 91.0)
- added B17C: , gen:15aef6ed4df9f5d238c1130cb8f0958fd2b96be76bbd888f3ba8bd3f59a98fb9, F.Cu at (164.4, 92.7)
- added B18C: , gen:15aef6ed4df9f5d238c1130cb8f0958fd2b96be76bbd888f3ba8bd3f59a98fb9, F.Cu at (161.6, 86.6)
- added B19C: , gen:15aef6ed4df9f5d238c1130cb8f0958fd2b96be76bbd888f3ba8bd3f59a98fb9, F.Cu at (166.1, 88.5)
- added B1C: , gen:15aef6ed4df9f5d238c1130cb8f0958fd2b96be76bbd888f3ba8bd3f59a98fb9, F.Cu at (120.0, 88.3)
- added B20C: , gen:15aef6ed4df9f5d238c1130cb8f0958fd2b96be76bbd888f3ba8bd3f59a98fb9, F.Cu at (180.7, 89.4)
- added B2C: , gen:15aef6ed4df9f5d238c1130cb8f0958fd2b96be76bbd888f3ba8bd3f59a98fb9, F.Cu at (134.7, 90.3)
- added B3C: , gen:15aef6ed4df9f5d238c1130cb8f0958fd2b96be76bbd888f3ba8bd3f59a98fb9, F.Cu at (140.1, 87.0)
- added B4C: , gen:15aef6ed4df9f5d238c1130cb8f0958fd2b96be76bbd888f3ba8bd3f59a98fb9, F.Cu at (137.4, 93.0)
- added B5C: , gen:15aef6ed4df9f5d238c1130cb8f0958fd2b96be76bbd888f3ba8bd3f59a98fb9, F.Cu at (142.8, 89.9)
- added B6C: , gen:15aef6ed4df9f5d238c1130cb8f0958fd2b96be76bbd888f3ba8bd3f59a98fb9, F.Cu at (140.2, 95.8)
- added D0U: , gen:537332067cad1e6cd91417ffa56b172e1694780f15a68609fbe58205aed1ad0e, F.Cu at (113.3, 84.3)
- added D1U: , gen:537332067cad1e6cd91417ffa56b172e1694780f15a68609fbe58205aed1ad0e, F.Cu at (109.7, 118.4)
- added D2U: , gen:537332067cad1e6cd91417ffa56b172e1694780f15a68609fbe58205aed1ad0e, F.Cu at (189.7, 118.5)
- added D3U: , gen:537332067cad1e6cd91417ffa56b172e1694780f15a68609fbe58205aed1ad0e, F.Cu at (186.3, 84.1)
- added ID0C: , gen:15aef6ed4df9f5d238c1130cb8f0958fd2b96be76bbd888f3ba8bd3f59a98fb9, F.Cu at (251.1, 147.1)
- added ID0J: , gen:95838f35713ea57911cd5ae6dd9bcb49a4c5df425079ab94d195f2c692cb5e30, F.Cu at (264.6, 147.6)
- added ID0L: , gen:c9032ee11626a7d8051c676e056ac92c83df9a1e8259cfacfdb10209d392f9d2, F.Cu at (137.1, 156.2)
- added ID0R: , gen:09d18632bfdd592ac9ac4d03ad983c1e61b79906e78d35a2a0c10d4ea1269f68, F.Cu at (254.7, 147.1)
- added ID1C: , gen:15aef6ed4df9f5d238c1130cb8f0958fd2b96be76bbd888f3ba8bd3f59a98fb9, F.Cu at (251.3, 148.1)
- added ID1J: , gen:95838f35713ea57911cd5ae6dd9bcb49a4c5df425079ab94d195f2c692cb5e30, F.Cu at (264.7, 147.9)
- added ID1L: , gen:c9032ee11626a7d8051c676e056ac92c83df9a1e8259cfacfdb10209d392f9d2, F.Cu at (146.5, 157.9)
- added ID1R: , gen:09d18632bfdd592ac9ac4d03ad983c1e61b79906e78d35a2a0c10d4ea1269f68, F.Cu at (254.8, 148.1)
- added ID2C: , gen:15aef6ed4df9f5d238c1130cb8f0958fd2b96be76bbd888f3ba8bd3f59a98fb9, F.Cu at (251.1, 149.1)
- added ID2J: , gen:95838f35713ea57911cd5ae6dd9bcb49a4c5df425079ab94d195f2c692cb5e30, F.Cu at (264.8, 148.3)
- added ID2L: , gen:c9032ee11626a7d8051c676e056ac92c83df9a1e8259cfacfdb10209d392f9d2, F.Cu at (155.1, 159.6)
- added ID2R: , gen:09d18632bfdd592ac9ac4d03ad983c1e61b79906e78d35a2a0c10d4ea1269f68, F.Cu at (254.9, 149.1)
- added ID3C: , gen:15aef6ed4df9f5d238c1130cb8f0958fd2b96be76bbd888f3ba8bd3f59a98fb9, F.Cu at (251.3, 149.9)
- added ID3J: , gen:95838f35713ea57911cd5ae6dd9bcb49a4c5df425079ab94d195f2c692cb5e30, F.Cu at (264.8, 148.6)
- added ID3L: , gen:c9032ee11626a7d8051c676e056ac92c83df9a1e8259cfacfdb10209d392f9d2, F.Cu at (166.2, 162.6)
- added ID3R: , gen:09d18632bfdd592ac9ac4d03ad983c1e61b79906e78d35a2a0c10d4ea1269f68, F.Cu at (254.9, 150.2)
- added ID4D: , gen:d30cd5d1ac2b05b3cbe32030fe258aa7b8dbe78edc4b93fc4c3e75fd2e28a25c, F.Cu at (245.1, 149.3)
- added ID5D: , gen:d30cd5d1ac2b05b3cbe32030fe258aa7b8dbe78edc4b93fc4c3e75fd2e28a25c, F.Cu at (245.2, 146.6)
- added ID6D: , gen:d30cd5d1ac2b05b3cbe32030fe258aa7b8dbe78edc4b93fc4c3e75fd2e28a25c, F.Cu at (245.5, 144.4)
- added ID7D: , gen:d30cd5d1ac2b05b3cbe32030fe258aa7b8dbe78edc4b93fc4c3e75fd2e28a25c, F.Cu at (245.5, 142.2)
- added IRT: , gen:09d18632bfdd592ac9ac4d03ad983c1e61b79906e78d35a2a0c10d4ea1269f68, F.Cu at (255.1, 136.2)
- added IU3C: , gen:15aef6ed4df9f5d238c1130cb8f0958fd2b96be76bbd888f3ba8bd3f59a98fb9, F.Cu at (249.8, 141.8)
- added T1U: , gen:5a2b29cdda025172b6c1938eb8323d0bef6bb00a32e80d3d8ab82bfb3852b84d, F.Cu at (118.4, 114.8)
- added T2U: , gen:5a2b29cdda025172b6c1938eb8323d0bef6bb00a32e80d3d8ab82bfb3852b84d, F.Cu at (181.4, 114.8)
- added vcc1_2_1U: , gen:00be09d7220a4ea10118fde02c68866a117403e6c69874da1578c3a54e2bd835, F.Cu at (114.3, 129.5)
- added vcc1_2_2U: , gen:00be09d7220a4ea10118fde02c68866a117403e6c69874da1578c3a54e2bd835, F.Cu at (177.8, 127.0)
- added vcc1_8U: , gen:8f6a8b6b5fb972609a253f1e69924482a5014d51fb3758bc278eca215963e1ec, F.Cu at (149.9, 50.8)
- added vcc1_8_1U: , gen:8f6a8b6b5fb972609a253f1e69924482a5014d51fb3758bc278eca215963e1ec, F.Cu at (91.4, 94.0)
- added vcc1_8_2U: , gen:8f6a8b6b5fb972609a253f1e69924482a5014d51fb3758bc278eca215963e1ec, F.Cu at (215.9, 106.7)
- added vcc2_8U: , gen:08e4b71c2dbcb779966d73d1978248ca96636087bbf1d4db6cf06e4ee0513d7c, F.Cu at (149.9, 58.5)
- added vcc3_0U: , gen:922a209d3ce6158d88552eee1f28af6afdf0641edad498ec0aae748706f5497b, F.Cu at (149.9, 66.1)
- added vcc3_0_1aU: , gen:922a209d3ce6158d88552eee1f28af6afdf0641edad498ec0aae748706f5497b, F.Cu at (91.4, 101.6)
- added vcc3_0_1bU: , gen:922a209d3ce6158d88552eee1f28af6afdf0641edad498ec0aae748706f5497b, F.Cu at (91.4, 109.2)
- added vcc3_0_2aU: , gen:922a209d3ce6158d88552eee1f28af6afdf0641edad498ec0aae748706f5497b, F.Cu at (215.9, 111.8)
- added vcc3_0_2bU: , gen:922a209d3ce6158d88552eee1f28af6afdf0641edad498ec0aae748706f5497b, F.Cu at (215.9, 116.8)
- B1, B10, B11, B15, B16, B17, B18, B19, B2, B20, B3, B4, B5, B6: footprint gen:d8f50a25e8aff35263f8cecdeff9c4e270c76c16c279eea1f2c61de037ffe0fa -> gen:fbc72c7906d62c511040786150c4aca9f7ffb0a6335083048829de2d171f3917; moved to F.Cu
- C1C10, C1C11, C1C12, C1C20, C1C21, C1C30, C1C31, C1C32, C1C33, C1C40, C1C41, C1C50, C1C51, C1C60, C1C61, C1C62, C1C63, C2C10, C2C11, C2C12, C2C20, C2C21, C2C30, C2C31, C2C32, C2C33, C2C40, C2C41, C2C50, C2C51, C2C60, C2C61, C2C62, C2C63, ID0C2, ID1C2, ID2C2, ID3C2, SC0, SC1, SC2, SC3, U2C0, U2C1, U2C10, U2C11, U2C2, U2C3, U2C4, U2C5, vcc1_2_2C1, vcc1_2_2C2, vcc1_8C1, vcc1_8C2, vcc1_8_1C1, vcc1_8_1C2, vcc1_8_2C1, vcc1_8_2C2, vcc2_8C1, vcc2_8C2, vcc3_0C1, vcc3_0C2, vcc3_0_1aC1, vcc3_0_1aC2, vcc3_0_1bC1, vcc3_0_1bC2, vcc3_0_2aC1, vcc3_0_2aC2, vcc3_0_2bC1, vcc3_0_2bC2: footprint gen:b8abd8cbc0b572999067c05d37fd407a90732e005a9769bc0f5d9b36d5f7537a -> gen:15aef6ed4df9f5d238c1130cb8f0958fd2b96be76bbd888f3ba8bd3f59a98fb9
- C1C70, C1C71, C2C70, C2C71: footprint gen:2dd82497e3d208e8bc654e5fd2889726ca886e84a8d673bd1d967596710ae728 -> gen:3af735041c9a949bfeabfb85bc7bf975c38b0916fa7e7388b3919d993ce08374
- C1FB1, C2FB1: footprint gen:4c7c45a8243ee1f12f8b92439e457e230f10814780b518cd649ab5c65f1663b6 -> gen:ebac41d1a35a3596bc713c11eee7f61d79ebc7743b0d7c28e1c9b0da10e2b7d7
- C1M1, C2M1: footprint gen:4d59d39d10787b911058ae9333354a532030edea4cb4e53179d64fabcbdb6f99 -> gen:df4eded634c017046067ccb08bbbdb0cd59e43cbc126ff0a3aedaa80e0e117e9
- C1R1, C1R2, C2R1, IR1, IR2, IR3: footprint gen:8b8e8cdd2a6c07e3e6c854f6b6a8f0d2287e4fa4909b824e776fd2ffcb4b4dd2 -> gen:09d18632bfdd592ac9ac4d03ad983c1e61b79906e78d35a2a0c10d4ea1269f68
- C1U1, C2U1: footprint gen:1ad7109002e715198f83cca1ffc9049c8e5399a3842da71963adabba6beed15b -> gen:8f3aa85955296813636e406510ac2cb44b6b28d253d1e3863a516e66fbc77376
- C2: footprint gen:96d8d9f3b01e3a213437eecc57d99723256313ff0fc11d8291488d1af641475f -> gen:8a6750ac66e1a6f76daf3ee494cac9e10424b63c23b0e42452ca9a9228b33a33; moved to F.Cu
- C2R2, R2: footprint gen:8b8e8cdd2a6c07e3e6c854f6b6a8f0d2287e4fa4909b824e776fd2ffcb4b4dd2 -> gen:09d18632bfdd592ac9ac4d03ad983c1e61b79906e78d35a2a0c10d4ea1269f68; moved to F.Cu
- ID0, ID1, ID2, ID3: footprint gen:c9b4f6ccae4bb0340b2ad5a6c71b1ffd2b7dd85978f603f30cef69603b532b8c -> gen:9c2b389c2dd7476cffe76adcd72a717edfd362f90df0b7c4d35bb2dfff612c12
- IU3: footprint gen:7f2b3144da42c433b15ca783ca7830c64f1f439c0eded0fed474f7f4b6ae4199 -> gen:cf30eca5ca4d85bf0ca83f28dce2ce8be3fb97701a118abd87ff880ab16f57bd; moved to F.Cu
- M0, M1, M2, M3: footprint gen:3c7f55a43bbd183404c5b8309475486c24daf5a9c2963092a0b256ddf24e95e1 -> gen:a2599a6c9388b85363dc78da9aac506bd81748babe4024ae1fcc4e8439878feb
- MU1: footprint gen:118301f00dc3a559b9b2dce5a7b5f72bf6d5ed1b69630a5bdce773a57167cb56 -> gen:88da571ed73d85986bd9b872487b21259fb0b9c897f7fa68810db8ac66ed3172
- P1: footprint gen:3f8ed9d7be0e74029e88378a59fbf78c1191c3dbd4709bec51884f93e57b519c -> gen:a1403a4ac11b1752655c81b77c786537d75d8acf64ea88171c3d4e9379b9cc3d
- SU1: footprint gen:f9c3ae8e9607776eb8d584f2f53baa49589c5cbd0e39654446d2f839acd0d9d0 -> gen:16ea7882d7f656d5472747c5083fa739ddb39b94832403c213f100a5ca75712f
- SU2: footprint gen:604093d92b23f96c780cabef8c052d038c2078bb1aa740e14df8b0cb48f3327f -> gen:3aa3b0dc59e4a041f536098cfce6f75865de9507baa2cfe5e0850a7ef365d386
- U2: footprint gen:37c349b4ccef9ca1e6dfa7e726c437006c67516ca70700a0b276a014844c8cb2 -> gen:08c9724177c4578a8ec67f3df913aab08fb61a69285502eb5c729cbf90cbdb19
- vcc1_2_1C1, vcc1_2_1C2: footprint gen:b8abd8cbc0b572999067c05d37fd407a90732e005a9769bc0f5d9b36d5f7537a -> gen:15aef6ed4df9f5d238c1130cb8f0958fd2b96be76bbd888f3ba8bd3f59a98fb9; moved to F.Cu
Connections:
- B1 pad 2: pair1N -> pair1P
- B1 pad 3: pair1P -> pair1N
- B1 pad 6: out1P -> out1N
- B1 pad 7: out1N -> out1P
- B10 pad 2: out10N -> out10P
- B10 pad 3: out10P -> out10N
- B10 pad 6: pair10P -> pair10N
- B10 pad 7: pair10N -> pair10P
- B11 pad 2: out11P -> out11N
- B11 pad 3: out11N -> out11P
- B11 pad 6: pair11N -> pair11P
- B11 pad 7: pair11P -> pair11N
- B15 pad 2: out15P -> out15N
- B15 pad 3: out15N -> out15P
- B15 pad 6: pair15N -> pair15P
- B15 pad 7: pair15P -> pair15N
- B16 pad 2: out16P -> out16N
- B16 pad 3: out16N -> out16P
- B16 pad 6: pair16N -> pair16P
- B16 pad 7: pair16P -> pair16N
- B17 pad 2: out17N -> out17P
- B17 pad 3: out17P -> out17N
- B17 pad 6: pair17P -> pair17N
- B17 pad 7: pair17N -> pair17P
- B18 pad 2: out18P -> out18N
- B18 pad 3: out18N -> out18P
- B18 pad 6: pair18N -> pair18P
- B18 pad 7: pair18P -> pair18N
- B19 pad 2: out19P -> out19N
- B19 pad 3: out19N -> out19P
- B19 pad 6: pair19N -> pair19P
- B19 pad 7: pair19P -> pair19N
- B2 pad 2: out2P -> out2N
- B2 pad 3: out2N -> out2P
- B2 pad 6: pair2N -> pair2P
- B2 pad 7: pair2P -> pair2N
- B20 pad 2: pair20P -> pair20N
- B20 pad 3: pair20N -> pair20P
- B20 pad 6: out20N -> out20P
- B20 pad 7: out20P -> out20N
- B3 pad 2: out3P -> out3N
- B3 pad 3: out3N -> out3P
- B3 pad 6: pair3N -> pair3P
- B3 pad 7: pair3P -> pair3N
- B4 pad 2: out4P -> out4N
- B4 pad 3: out4N -> out4P
- B4 pad 6: pair4N -> pair4P
- B4 pad 7: pair4P -> pair4N
- B5 pad 2: out5N -> out5P
- B5 pad 3: out5P -> out5N
- B5 pad 6: pair5P -> pair5N
- B5 pad 7: pair5N -> pair5P
- B6 pad 2: out6N -> out6P
- B6 pad 3: out6P -> out6N
- B6 pad 6: pair6P -> pair6N
- B6 pad 7: pair6N -> pair6P
Routing:
- net gnd: track 64.6 -> 79.2 mm, vias 66 -> 74
- net T2SCLK: track 13.2 -> 3.08 mm, vias 2 -> 0
- net vcc3_3in: track 25.4 -> 16.0 mm
- net C2vdd_pix: track 2.74 -> 0.49 mm, vias 2 -> 1
- net out19N: track 23.6 -> 21.6 mm, vias 1 -> 2
- net out19P: track 23.3 -> 21.5 mm, vias 1 -> 2
- net _B11_5_NC: track 0.00 -> 1.46 mm
- net _B3_5_NC: track 0.00 -> 1.23 mm
- net _B5_5_NC: track 0.00 -> 0.96 mm
- net _B1_5_NC: track 0.00 -> 0.90 mm
- net _B17_5_NC: track 0.00 -> 0.90 mm
- net _B10_5_NC: track 0.00 -> 0.90 mm
- net _B4_5_NC: track 0.00 -> 0.85 mm
- net _B6_5_NC: track 0.00 -> 0.81 mm
- net _B2_5_NC: track 0.00 -> 0.79 mm
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