File: pcb/camera2/kicad/camera2.kicad_pcb (KiCad board)
At the start: 4 copper layers, 96.5 x 45.7 mm, 172 parts

Commit message: work
Parts:
- removed the ID4D at (245.1, 149.3)
- removed the ID5D at (245.2, 146.6)
- removed the ID6D at (245.5, 144.4)
- removed the ID7D at (245.5, 142.2)
- removed the vcc1_2_1U at (114.3, 129.5)
- removed the vcc1_2_2U at (177.8, 127.0)
- removed the vcc1_8U at (149.9, 50.8)
- removed the vcc1_8_1U at (91.4, 94.0)
- removed the vcc1_8_2U at (215.9, 106.7)
- removed the vcc2_8U at (149.9, 58.5)
- removed the vcc3_0U at (149.9, 66.1)
- removed the vcc3_0_1aU at (91.4, 101.6)
- removed the vcc3_0_1bU at (91.4, 109.2)
- removed the vcc3_0_2aU at (215.9, 111.8)
- removed the vcc3_0_2bU at (215.9, 116.8)
- added ID4D: , gen:736f40deae4fa0d46eb981f73fc34307d5e4f1c6ef1d3d54b3ef8bd5433cf1fa, F.Cu at (245.1, 149.3)
- added ID5D: , gen:736f40deae4fa0d46eb981f73fc34307d5e4f1c6ef1d3d54b3ef8bd5433cf1fa, F.Cu at (245.2, 146.6)
- added ID6D: , gen:736f40deae4fa0d46eb981f73fc34307d5e4f1c6ef1d3d54b3ef8bd5433cf1fa, F.Cu at (245.5, 144.4)
- added ID7D: , gen:736f40deae4fa0d46eb981f73fc34307d5e4f1c6ef1d3d54b3ef8bd5433cf1fa, F.Cu at (245.5, 142.2)
- added vcc1_2_1U: , gen:69356af040f643a03a60cd7bc275e3a7b7db7b36bedbc785edf210b2af987edd, B.Cu at (117.8, 116.8)
- added vcc1_2_2U: , gen:69356af040f643a03a60cd7bc275e3a7b7db7b36bedbc785edf210b2af987edd, B.Cu at (180.8, 116.9)
- added vcc1_8U: , gen:dd290dda99227062545065e61da3a294210741383d6626792b429e6518dce39b, F.Cu at (149.9, 50.8)
- added vcc1_8_1U: , gen:dd290dda99227062545065e61da3a294210741383d6626792b429e6518dce39b, F.Cu at (91.4, 94.0)
- added vcc1_8_2U: , gen:dd290dda99227062545065e61da3a294210741383d6626792b429e6518dce39b, F.Cu at (215.9, 106.7)
- added vcc2_8U: , gen:a8b18f1694ca75820e6cb9a3a465c2602d11b606d4cb71bafed472bb199c8d3b, F.Cu at (149.9, 58.5)
- added vcc3_0U: , gen:6f747c56d74b7a0e3aabdf61657f08e040c4918040aef088c9db2b0a015cfaee, F.Cu at (149.9, 66.1)
- added vcc3_0_1aU: , gen:6f747c56d74b7a0e3aabdf61657f08e040c4918040aef088c9db2b0a015cfaee, F.Cu at (91.4, 101.6)
- added vcc3_0_1bU: , gen:6f747c56d74b7a0e3aabdf61657f08e040c4918040aef088c9db2b0a015cfaee, F.Cu at (91.4, 109.2)
- added vcc3_0_2aU: , gen:6f747c56d74b7a0e3aabdf61657f08e040c4918040aef088c9db2b0a015cfaee, F.Cu at (215.9, 111.8)
- added vcc3_0_2bU: , gen:6f747c56d74b7a0e3aabdf61657f08e040c4918040aef088c9db2b0a015cfaee, F.Cu at (215.9, 116.8)
- B1, B10, B11, B15, B16, B17, B18, B19, B2, B20, B3, B4, B5, B6: footprint gen:fbc72c7906d62c511040786150c4aca9f7ffb0a6335083048829de2d171f3917 -> gen:ec4c19d9976d47b7fe720a0af2fbe08b743ab89b55bf072d08ff9279dcf65392
- IU3: footprint gen:cf30eca5ca4d85bf0ca83f28dce2ce8be3fb97701a118abd87ff880ab16f57bd -> gen:10055cda59e5a70ce0bc86550a5f75ef499931ada32159cd6aabb90b37b327da
- MU1: footprint gen:88da571ed73d85986bd9b872487b21259fb0b9c897f7fa68810db8ac66ed3172 -> gen:26b7ea9bab8162176cb957c507b2d408ca1ea6a8e21ee01cd2df422f221d0556
- vcc1_2_1C1, vcc1_2_1C2, vcc1_2_2C1, vcc1_2_2C2: moved to B.Cu
- moved ID3L 44.2 mm to (166.9, 118.4)
- moved ID2L 41.4 mm to (158.4, 118.2)
- moved ID1L 40.0 mm to (140.7, 118.4)
- moved ID0L 38.5 mm to (132.7, 118.0)
- moved U2C1 17.4 mm to (157.1, 114.0), turned to 0 degrees
- moved vcc1_2_1C1 15.4 mm to (120.4, 116.8), turned to 270 degrees
- moved vcc1_2_2C1 12.9 mm to (183.3, 116.8)
- moved U2C5 12.6 mm to (160.4, 109.8), turned to 45 degrees
- moved vcc1_2_1C2 11.9 mm to (115.4, 117.7), turned to 270 degrees
- moved U2C10 10.8 mm to (140.7, 111.9), turned to 180 degrees
- moved vcc1_2_2C2 9.60 mm to (178.4, 117.6)
- moved U2C3 7.64 mm to (138.7, 108.5)
- moved U2C0 6.09 mm to (142.8, 101.9)
- moved U2C2 5.64 mm to (153.4, 98.2), turned to 90 degrees
- moved U2C11 5.25 mm to (148.8, 96.7)
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Connections:
- U2 pad 1: _U2_1_IO2_1 -> C2MISO
- U2 pad 10: _U2_10_IO2_10 -> C2trigger0
- U2 pad 12: pair14N -> _U2_12_IO2_12
- U2 pad 13: pair14P -> _U2_13_IO2_13
- U2 pad 14: pair13N -> _U2_14_IO1_14
- U2 pad 15: pair13P -> _U2_15_IO1_15
- U2 pad 16: pair12P -> _U2_16_IO1_16
- U2 pad 17: pair12N -> pair14N
- U2 pad 18: pair9N -> pair14P
- U2 pad 19: pair9P -> pair13N
- U2 pad 2: _U2_2_IO2_2 -> C2MOSI
- U2 pad 22: pair8P -> pair13P
- U2 pad 23: pair8N -> pair12P
- U2 pad 24: pair7P -> pair12N
- U2 pad 27: pair7N -> pair9N
- U2 pad 28: C1SCLK -> pair9P
- U2 pad 29: C1MISO -> pair8P
- U2 pad 3: _U2_3_IO2_3 -> C2_ss_n
- U2 pad 30: C1MOSI -> pair8N
- U2 pad 32: C1_ss_n -> pair7P
- U2 pad 33: C1reset_n -> pair7N
- U2 pad 34: C1monitor1 -> _U2_34_IO1_34
- U2 pad 35: C1monitor0 -> _U2_35_IO1_35
- U2 pad 36: C1trigger2 -> _U2_36_IO1_36
- U2 pad 37: C1trigger1 -> _U2_37_IO1_37
- U2 pad 39: C1trigger0 -> C1SCLK
- U2 pad 4: _U2_4_IO2_4 -> C2reset_n
- U2 pad 40: T1_master_clk -> C1MISO
- U2 pad 41: T1_pwr_dwn_l -> C1MOSI
- U2 pad 42: T1_reset_l -> C1_ss_n
- U2 pad 43: T1SCL -> C1reset_n
- U2 pad 44: T1SDA -> C1monitor1
- U2 pad 46: T1MOSI -> C1monitor0
- U2 pad 49: T1MISO -> C1trigger2
- U2 pad 50: T1SCLK -> C1trigger1
- U2 pad 52: T1_ss_n -> C1trigger0
- U2 pad 53: temp_bus -> T1_master_clk
- U2 pad 54: led_pwm0 -> T1_pwr_dwn_l
- U2 pad 55: led_pwm1 -> T1_reset_l
- U2 pad 56: led_pwm2 -> T1SCL
- U2 pad 58: led_pwm3 -> T1SDA
- U2 pad 59: led_nSHDN -> T1MOSI
- U2 pad 6: _U2_6_IO2_6 -> C2monitor1
- U2 pad 60: _U2_60_IO1_60 -> T1MISO
- U2 pad 61: _U2_61_IO1_61 -> T1SCLK
- U2 pad 63: _U2_63_IO1_63 -> T1_ss_n
- U2 pad 7: _U2_7_IO2_7 -> C2monitor0
- U2 pad 77: T2SCL -> _U2_77_IO2_77
- U2 pad 78: T2SDA -> _U2_78_IO2_78
- U2 pad 79: T2MOSI -> _U2_79_IO2_79
- U2 pad 8: _U2_8_IO2_8 -> C2trigger2
- U2 pad 80: T2MISO -> _U2_80_IO2_80
- U2 pad 81: T2SCLK -> _U2_81_IO2_81
- U2 pad 82: T2_ss_n -> _U2_82_IO2_82
- U2 pad 85: T2_master_clk -> _U2_85_IO2_85
- U2 pad 86: T2_pwr_dwn_l -> _U2_86_IO2_86
- U2 pad 87: T2_reset_l -> _U2_87_IO2_87
- U2 pad 89: C2SCLK -> T2SCL
- U2 pad 9: _U2_9_IO2_9 -> C2trigger1
- U2 pad 90: C2MISO -> T2SDA
- U2 pad 91: C2MOSI -> T2MOSI
- U2 pad 92: C2_ss_n -> T2MISO
- U2 pad 93: C2reset_n -> T2SCLK
- U2 pad 94: C2monitor1 -> T2_ss_n
- U2 pad 95: C2monitor0 -> T2_master_clk
- U2 pad 96: C2trigger2 -> T2_pwr_dwn_l
- U2 pad 97: C2trigger1 -> T2_reset_l
- U2 pad 99: C2trigger0 -> C2SCLK
Routing:
- net T2SCLK: track 3.08 -> 31.7 mm, vias 0 -> 2
- net C1monitor1: track 2.90 -> 29.4 mm
- net C1monitor0: track 3.27 -> 29.6 mm
- net C1reset_n: track 2.54 -> 28.7 mm
- net C1_ss_n: track 2.19 -> 27.9 mm
- net C1trigger2: track 3.55 -> 29.0 mm
- net C1trigger0: track 8.06 -> 33.2 mm
- net C1trigger1: track 5.45 -> 30.5 mm
- net C1MOSI: track 1.80 -> 25.2 mm
- net C1MISO: track 1.45 -> 24.5 mm
- net C1SCLK: track 1.11 -> 23.7 mm
- net T2SCL: track 28.0 -> 48.4 mm
- net T2SDA: track 28.3 -> 48.7 mm
- net T2MOSI: track 14.5 -> 34.7 mm
- net T2MISO: track 15.3 -> 35.5 mm
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Other:
- board text added: "move clock in buffers to be with others"
