File: pcb/camera2/kicad/camera2.kicad_pcb (KiCad board)
At the start: 4 copper layers, 96.5 x 45.7 mm, 173 parts

Commit message: prev
Parts:
- removed the ID4D at (245.1, 149.3)
- removed the ID5D at (245.2, 146.6)
- removed the ID6D at (245.5, 144.4)
- removed the ID7D at (245.5, 142.2)
- removed the vcc1_2_1U at (117.8, 116.8)
- removed the vcc1_2_2U at (180.8, 116.9)
- removed the vcc1_8U at (144.7, 108.1)
- removed the vcc1_8_1U at (91.4, 94.0)
- removed the vcc1_8_2U at (185.9, 100.6)
- removed the vcc2_8U at (149.9, 58.5)
- removed the vcc3_0U at (153.7, 108.2)
- removed the vcc3_0_1aU at (91.4, 101.6)
- removed the vcc3_0_1bU at (91.4, 109.2)
- removed the vcc3_0_2aU at (185.7, 93.0)
- removed the vcc3_0_2bU at (179.6, 95.5)
- added IC1: , gen:15aef6ed4df9f5d238c1130cb8f0958fd2b96be76bbd888f3ba8bd3f59a98fb9, F.Cu at (234.8, 142.8)
- added ID4D: , gen:b02a108efab3f2a1a80b6c611792ba31b89791d9e4fe9f59408e818a7abde35f, F.Cu at (238.0, 154.8)
- added ID5D: , gen:b02a108efab3f2a1a80b6c611792ba31b89791d9e4fe9f59408e818a7abde35f, F.Cu at (236.0, 154.8)
- added ID6D: , gen:b02a108efab3f2a1a80b6c611792ba31b89791d9e4fe9f59408e818a7abde35f, F.Cu at (234.0, 154.8)
- added ID7D: , gen:b02a108efab3f2a1a80b6c611792ba31b89791d9e4fe9f59408e818a7abde35f, F.Cu at (232.0, 154.8)
- added vcc1_2_1U: , gen:d4799acb2780d1093158ca020a5a853254575767f1cc4480606e32db94928da4, B.Cu at (117.8, 116.8)
- added vcc1_2_2U: , gen:d4799acb2780d1093158ca020a5a853254575767f1cc4480606e32db94928da4, B.Cu at (180.8, 116.9)
- added vcc1_8U: , gen:de1936faee739f8d943353fa792e70468b5c635e00572ad49399fbe3d51d34e6, B.Cu at (144.7, 108.1)
- added vcc1_8_1U: , gen:de1936faee739f8d943353fa792e70468b5c635e00572ad49399fbe3d51d34e6, F.Cu at (91.4, 94.0)
- added vcc1_8_2U: , gen:de1936faee739f8d943353fa792e70468b5c635e00572ad49399fbe3d51d34e6, B.Cu at (185.9, 100.6)
- added vcc2_8U: , gen:feaf106ac02cf50d222dd4be3a9280b8cefde7375b17b7c74366abb482f061a3, F.Cu at (149.9, 58.5)
- added vcc3_0U: , gen:458d1a0a0e97a12f0c2522c3927ea8716f002d7a906540b8d07400dd828608d8, B.Cu at (153.7, 108.2)
- added vcc3_0_1aU: , gen:458d1a0a0e97a12f0c2522c3927ea8716f002d7a906540b8d07400dd828608d8, F.Cu at (91.4, 101.6)
- added vcc3_0_1bU: , gen:458d1a0a0e97a12f0c2522c3927ea8716f002d7a906540b8d07400dd828608d8, F.Cu at (91.4, 109.2)
- added vcc3_0_2aU: , gen:458d1a0a0e97a12f0c2522c3927ea8716f002d7a906540b8d07400dd828608d8, B.Cu at (185.7, 93.0)
- added vcc3_0_2bU: , gen:458d1a0a0e97a12f0c2522c3927ea8716f002d7a906540b8d07400dd828608d8, B.Cu at (179.6, 95.5)
- B1, B10, B11, B15, B16, B17, B18, B19, B2, B20, B3, B4, B5, B6: footprint gen:d5d747658d1f210c64ba5afe5344e053b8a2d55b6f3d730df7e8fcb94f698341 -> gen:8f814f70c313fe4864baf07274623f11be704aa44e6ea7b08be35d28071a1cc9
- C1C21: moved to B.Cu
- C1U1, C2U1: footprint gen:2c43dbd9f6af1bb8faf0dc21f50b99c6562a4598033a204bce2cbb3aa0ac77e0 -> gen:8a0fe1e2c65c1147e75bc2bf912fd2f2d0a71d7fb4e393d72bdb606ffdff7ec6
- IU3: footprint gen:3cf7be2816aebb87938a72439acbc299fb39ba3576f28d4585b83a929bdf084e -> gen:076c46a950db2b0d12b3618cb5aa6e3a9d0ff0f63186aeba8efe585542761209
- MU1: footprint gen:090464809685175b38cabe7209672ac088d3c8d16318e2135ae4ec4fabcf0fdf -> gen:fe677413a6f5da87e344f01776feb477e53f3e2ebb255b293112f82b9e19914e
- P2: footprint gen:241492fd899311e7d9c7e61eadc180b241cdf3d88f3ef5a7a5d9a913c8bb5d54 -> gen:fac2a339cebc6f442379fe0f57132eb50ea48522eb26f51410436de4a1288066
- moved SU1 98.7 mm to (175.5, 61.1), turned to 45 degrees
- moved ID2C2 29.0 mm to (229.8, 147.5), turned to 180 degrees
- moved ID3C2 26.9 mm to (232.2, 144.8), turned to 90 degrees
- moved IR3 22.3 mm to (229.8, 150.0)
- moved IU3 22.0 mm to (235.0, 149.0)
- moved ID0C 21.7 mm to (234.1, 160.6)
- moved ID1C 21.7 mm to (234.3, 161.6)
- moved ID2C 21.7 mm to (234.1, 162.6)
- moved ID3C 21.7 mm to (234.3, 163.4)
- moved IRT 21.6 mm to (235.2, 144.8)
- moved ID0C2 20.4 mm to (237.8, 144.8), turned to 90 degrees
- moved ID1C2 18.1 mm to (240.2, 147.5)
- moved SU2 14.2 mm to (100.7, 62.4), turned to 45 degrees
- moved IU3C 12.6 mm to (240.2, 150.0), turned to 0 degrees
- moved ID0R 12.0 mm to (255.5, 159.0), turned to 270 degrees
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Connections:
- ID0C pad 1: Icap0 -> vcc5in
- ID1C pad 1: Icap1 -> vcc5in
- ID2C pad 1: Icap2 -> vcc5in
- ID3C pad 1: Icap3 -> vcc5in
- IU3 pad 19: _IU3_19_NC -> gnd
- IU3 pad 20: _IU3_20_NC -> gnd
- IU3 pad 21: _IU3_21_NC -> gnd
- IU3 pad 30: _IU3_30_NC -> gnd
- IU3 pad 31: _IU3_31_NC -> gnd
- IU3 pad 32: _IU3_32_NC -> gnd
Routing:
- net C1MOSI: track 4.56 -> 25.2 mm
- net vcc1_8: track 9.81 -> 21.5 mm, vias 1 -> 2
- net gnd: track 124.3 -> 134.1 mm, vias 115 -> 116
- net vcc3_0_1a: track 0.00 -> 7.49 mm
- net vcc3_0_2a: track 1.22 -> 6.16 mm
- net C1vdd_pix: track 0.00 -> 4.79 mm
- net C2vdd_pix: track 0.00 -> 4.79 mm
- net vcc1_8_1: track 0.00 -> 3.95 mm
- net vcc1_8_2: track 2.51 -> 5.89 mm
- net Iref: track 0.00 -> 3.28 mm
- net C1_ss_n: track 27.9 -> 29.4 mm
- net vcc3_0: track 15.7 -> 17.0 mm
- net Irt: track 0.00 -> 1.25 mm
- net pair12N: track 20.4 -> 19.9 mm
- added copper zone on F.Cu, net Isw0
- added copper zone on F.Cu, net Isw1
- added copper zone on F.Cu, net Isw2
- added copper zone on F.Cu, net Isw3

Commit message: more routing
Parts:
- removed the ID4D at (238.0, 154.8)
- removed the ID5D at (236.0, 154.8)
- removed the ID6D at (234.0, 154.8)
- removed the ID7D at (232.0, 154.8)
- removed the vcc1_2_1U at (117.8, 116.8)
- removed the vcc1_2_2U at (180.8, 116.9)
- removed the vcc1_8U at (144.7, 108.1)
- removed the vcc1_8_1U at (91.4, 94.0)
- removed the vcc1_8_2U at (185.9, 100.6)
- removed vcc2_8C1, vcc2_8C2: , gen:15aef6ed4df9f5d238c1130cb8f0958fd2b96be76bbd888f3ba8bd3f59a98fb9
- removed vcc2_8U: , gen:feaf106ac02cf50d222dd4be3a9280b8cefde7375b17b7c74366abb482f061a3
- removed the vcc3_0U at (153.7, 108.2)
- removed the vcc3_0_1aU at (91.4, 101.6)
- removed the vcc3_0_1bU at (91.4, 109.2)
- removed the vcc3_0_2aU at (185.7, 93.0)
- removed the vcc3_0_2bU at (179.6, 95.5)
- added ID4D: , gen:e3580ea2dbc098b2a536e874046aaf6f7ebd313d69432f15c77bc45374301d07, F.Cu at (238.0, 154.8)
- added ID5D: , gen:e3580ea2dbc098b2a536e874046aaf6f7ebd313d69432f15c77bc45374301d07, F.Cu at (236.0, 154.8)
- added ID6D: , gen:e3580ea2dbc098b2a536e874046aaf6f7ebd313d69432f15c77bc45374301d07, F.Cu at (234.0, 154.8)
- added ID7D: , gen:e3580ea2dbc098b2a536e874046aaf6f7ebd313d69432f15c77bc45374301d07, F.Cu at (232.0, 154.8)
- added vcc1_2_1U: , gen:6c14373226c8db886f922428da15573c84e66209c7d58ce547ef9f04c698a19f, B.Cu at (118.1, 116.8)
- added vcc1_2_2U: , gen:6c14373226c8db886f922428da15573c84e66209c7d58ce547ef9f04c698a19f, B.Cu at (181.0, 116.8)
- added vcc1_8U: , gen:cea7e99fe6780f55b5f4124ae3c472ad09a8cea9fb4f8090fbcb898114cf92fd, B.Cu at (144.7, 108.1)
- added vcc1_8_1U: , gen:cea7e99fe6780f55b5f4124ae3c472ad09a8cea9fb4f8090fbcb898114cf92fd, B.Cu at (91.4, 94.0)
- added vcc1_8_2U: , gen:cea7e99fe6780f55b5f4124ae3c472ad09a8cea9fb4f8090fbcb898114cf92fd, B.Cu at (185.9, 100.6)
- added vcc2_8_1C1: , gen:15aef6ed4df9f5d238c1130cb8f0958fd2b96be76bbd888f3ba8bd3f59a98fb9, B.Cu at (115.6, 113.0)
- added vcc2_8_1C2: , gen:15aef6ed4df9f5d238c1130cb8f0958fd2b96be76bbd888f3ba8bd3f59a98fb9, B.Cu at (120.7, 113.0)
- added vcc2_8_1U: , gen:20a1bec42615eb95c327f6c4bbbe16c066c1745dadaaaae28f387ebf38620350, B.Cu at (118.1, 113.0)
- added vcc2_8_2C1: , gen:15aef6ed4df9f5d238c1130cb8f0958fd2b96be76bbd888f3ba8bd3f59a98fb9, B.Cu at (179.1, 113.0)
- added vcc2_8_2C2: , gen:15aef6ed4df9f5d238c1130cb8f0958fd2b96be76bbd888f3ba8bd3f59a98fb9, B.Cu at (184.2, 113.0)
- added vcc2_8_2U: , gen:20a1bec42615eb95c327f6c4bbbe16c066c1745dadaaaae28f387ebf38620350, B.Cu at (181.6, 113.0)
- added vcc3_0U: , gen:2547c2f8ec5c0fd3b3ffe65b36caba8ac885a0357d6a1f4e7a71534fd4946663, B.Cu at (153.7, 108.2)
- added vcc3_0_1aU: , gen:2547c2f8ec5c0fd3b3ffe65b36caba8ac885a0357d6a1f4e7a71534fd4946663, B.Cu at (91.4, 101.6)
- added vcc3_0_1bU: , gen:2547c2f8ec5c0fd3b3ffe65b36caba8ac885a0357d6a1f4e7a71534fd4946663, B.Cu at (91.4, 109.2)
- added vcc3_0_2aU: , gen:2547c2f8ec5c0fd3b3ffe65b36caba8ac885a0357d6a1f4e7a71534fd4946663, B.Cu at (185.7, 93.0)
- added vcc3_0_2bU: , gen:2547c2f8ec5c0fd3b3ffe65b36caba8ac885a0357d6a1f4e7a71534fd4946663, B.Cu at (179.6, 95.5)
- B1, B10, B11, B15, B16, B17, B18, B19, B2, B20, B3, B4, B5, B6: footprint gen:8f814f70c313fe4864baf07274623f11be704aa44e6ea7b08be35d28071a1cc9 -> gen:5177976ce074159293d06658834db7fd460ac52f9f70d3076b2631a81124ed6d
- C1U1, C2U1: footprint gen:8a0fe1e2c65c1147e75bc2bf912fd2f2d0a71d7fb4e393d72bdb606ffdff7ec6 -> gen:6530bc05c16df6db2c9c4ca17d553006c6430797659c6299eea2475f90c9972e
- IU3: footprint gen:076c46a950db2b0d12b3618cb5aa6e3a9d0ff0f63186aeba8efe585542761209 -> gen:b92df038f4aee81fe2e33c8b61062eab4c628e367988fedf188c2dbfd3584f77
- MU1: footprint gen:fe677413a6f5da87e344f01776feb477e53f3e2ebb255b293112f82b9e19914e -> gen:ea86113c9ec2dff1a068f9ae0d02d564a2ae5741c070a78799bd725783cf0f0a
- P2: footprint gen:fac2a339cebc6f442379fe0f57132eb50ea48522eb26f51410436de4a1288066 -> gen:3442744b53b14b6ffd8ec656ce035acacb2313dc3b469232c1468ad8224701f6
- vcc1_8_1C1, vcc1_8_1C2, vcc3_0_1aC1, vcc3_0_1aC2, vcc3_0_1bC1, vcc3_0_1bC2: moved to B.Cu
- moved vcc1_2_1C2 0.87 mm to (115.6, 116.8)
- moved D2U 0.38 mm to (190.1, 118.5)
- moved D0U 0.33 mm to (113.3, 83.9)
- moved vcc1_2_1C1 0.26 mm to (120.7, 116.8)
- moved vcc1_2_2C1 0.23 mm to (183.5, 116.8)
- moved D3U 0.22 mm to (186.4, 83.9)
- moved ID0L 0.13 mm to (132.7, 118.1)
- moved vcc1_2_2C2 0.13 mm to (178.4, 117.5)
- moved D1U 0.11 mm to (109.6, 118.5)
- turned SU1 to 90 degrees
- turned vcc1_8_1C1 to 90 degrees
- turned vcc1_8_1C2 to 90 degrees
- turned vcc3_0_1aC1 to 90 degrees
- turned vcc3_0_1aC2 to 90 degrees
- turned vcc3_0_1bC1 to 90 degrees
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Connections:
- IU3 pad 14: Ivadj3 -> Irefdiv
- IU3 pad 15: Ivadj2 -> Irefdiv
- IU3 pad 36: Ivadj1 -> Irefdiv
- IU3 pad 37: Ivadj0 -> Irefdiv
- T1U pad 19: vcc2_8 -> vcc2_8_1
- T2U pad 19: vcc2_8 -> vcc2_8_2
Routing:
- net vcc3_3in: track 34.3 -> 90.6 mm, vias 15 -> 22
- net gnd: track 134.1 -> 167.0 mm, vias 116 -> 135
- net vcc2_8_1: track 0.00 -> 5.32 mm, vias 0 -> 1
- net vcc2_8_2: track 0.00 -> 5.11 mm, vias 0 -> 1
- net vcc1_2_1: track 0.66 -> 3.28 mm
- net vcc1_2_2: track 0.65 -> 3.14 mm
- net vcc2_8: track 1.31 -> 0.00 mm, vias 2 -> 0

Commit message: more routing
Parts:
- moved SU1 98.7 mm to (76.8, 58.6), turned to 0 degrees
- moved SU2 6.46 mm to (94.3, 61.6), turned to 180 degrees
Routing:
- net vcc3_3in: track 90.6 -> 98.5 mm, vias 22 -> 23
- net temp_bus: track 0.00 -> 3.91 mm, vias 0 -> 4
- net gnd: track 167.0 -> 170.1 mm, vias 135 -> 136
